Commit message: added all the sensors

File: description/robot.urdf.xacro (robot description, xacro)
@@ -3,3 +3,6 @@
     <xacro:include filename="robot_core.xacro"/>
     <xacro:include filename="gazebo_include.xacro"/>
+    <xacro:include filename="lidar.xacro"/>
+    <!-- <xacro:include filename="camera.xacro"/> -->
+    <xacro:include filename="depth_camera.xacro"/>
 </robot>

File: description/robot_core.xacro (robot description, xacro)
@@ -14,4 +14,7 @@
     <material name="blue">
         <color rgba="0.2 0.2 1 1"/>
+    </material>
+    <material name="red">
+        <color rgba="1 0.2 0.2 1"/>
     </material>
     <!-- LINKS AND JOINTS -->
@@ -58,5 +61,5 @@
             <origin xyz="0 0 0"/>
         </visual>
-         <collision>
+        <collision>
             <geometry>
                 <cylinder radius="0.050" length="0.040"/>
